Commit message: updated urdf files

File: urdf/digitwin.urdf.xacro (robot description, xacro)
@@ -1,3 +1,2 @@
-<?xml version="1.0"?>
 <robot xmlns:xacro="http://www.ros.org/wiki/xacro" name="twin">
     <material name="gray">
@@ -30,5 +29,5 @@
     <link name="world"> </link>
     <joint name="world_to_table" type="fixed">
-        <origin xyz="0 0 0" rpy="1.5708 0 0"/>
+        <origin xyz="1 0 0" rpy="1.5708 0 0"/>
         <parent link="world"/>
         <child link="table"/>
@@ -36,5 +35,5 @@
     <link name="table">
         <visual>
-            <origin xyz="1 0 0" rpy="0 0 0"/>
+            <origin xyz="2 0 0" rpy="0 0 0"/>
             <geometry>
                 <box size="5 0.1 3"/>
@@ -50,5 +49,5 @@
     </link>
     <joint name="table_to_firstFloor" type="prismatic">
-        <origin xyz="0 0 0" rpy="0 0 0"/>
+        <origin xyz="0 0.25 0" rpy="0 0 0"/>
         <parent link="table"/>
         <child link="firstFloor"/>
@@ -72,5 +71,5 @@
     </link>
     <joint name="firstFloor_to_secondFloor" type="prismatic">
-        <origin xyz="0 0 0" rpy="0 0 0"/>
+        <origin xyz="0 0.25 0" rpy="0 0 0"/>
         <parent link="firstFloor"/>
         <child link="secondFloor"/>
@@ -94,5 +93,5 @@
     </link>
     <joint name="secondFloor_to_thirdFloor" type="prismatic">
-        <origin xyz="0 0 0" rpy="0 0 0"/>
+        <origin xyz="0 0.25 0" rpy="0 0 0"/>
         <parent link="secondFloor"/>
         <child link="thirdFloor"/>
@@ -116,5 +115,5 @@
     </link>
     <joint name="thirdFloor_to_fourthFloor" type="prismatic">
-        <origin xyz="0 0 0" rpy="0 0 0"/>
+        <origin xyz="0 0.25 0" rpy="0 0 0"/>
         <parent link="thirdFloor"/>
         <child link="fourthFloor"/>
@@ -138,5 +137,5 @@
     </link>
     <joint name="fourthFloor_to_fifthFloor" type="prismatic">
-        <origin xyz="0 0 0" rpy="0 0 0"/>
+        <origin xyz="0 0.25 0" rpy="0 0 0"/>
         <parent link="fourthFloor"/>
         <child link="fifthFloor"/>
@@ -162,5 +161,5 @@
         <parent link="world"/>
         <child link="camera"/>
-        <origin xyz="5 6 0" rpy="0 0 0"/>
+        <origin xyz="1 1 0" rpy="0 0 0"/>
     </joint>
     <link name="camera">

Commit message: updated urdf-fixed

File: urdf/digitwin.urdf.xacro (robot description, xacro)
@@ -29,5 +29,5 @@
     <link name="world"> </link>
     <joint name="world_to_table" type="fixed">
-        <origin xyz="1 0 0" rpy="1.5708 0 0"/>
+        <origin xyz="1 0 0" rpy="0 0 0"/>
         <parent link="world"/>
         <child link="table"/>
@@ -35,7 +35,7 @@
     <link name="table">
         <visual>
-            <origin xyz="2 0 0" rpy="0 0 0"/>
+            <origin xyz="0 0 0" rpy="0 0 0"/>
             <geometry>
-                <box size="5 0.1 3"/>
+                <box size="2 2 0.1"/>
             </geometry>
             <material name="gray"/>
@@ -44,115 +44,120 @@
             <origin xyz="1 0 0" rpy="0 0 0"/>
             <geometry>
-                <box size="5 0.1 3"/>
+                <box size="2 2 0.1"/>
             </geometry>
         </collision>
     </link>
+    <!-- Joint for stacking the floors vertically and allowing horizontal movement -->
     <joint name="table_to_firstFloor" type="prismatic">
-        <origin xyz="0 0.25 0" rpy="0 0 0"/>
+        <origin xyz="0 0 0.1" rpy="0 0 0"/> <!-- Positioning first floor directly on the table -->
         <parent link="table"/>
         <child link="firstFloor"/>
-        <axis xyz="1 0 0"/> <!-- Allows horizontal motion along the x-axis -->
+        <axis xyz="1 0 0"/> <!-- Horizontal movement along the x-axis -->
         <limit lower="-1.0" upper="1.0" effort="1000" velocity="1.0"/>
     </joint>
     <link name="firstFloor">
         <visual>
-            <origin xyz="0 0 0" rpy="0 0 0"/>
+            <origin xyz="0 0 1" rpy="0 0 0"/>
             <geometry>
-                <box size="1 2 1"/>
+                <box size="1 1 2"/>
             </geometry>
-            <material name="magenta"/>
+            <material name="red"/> <!-- Color changed to red -->
         </visual>
         <collision>
             <origin xyz="0 0 0" rpy="0 0 0"/>
             <geometry>
-                <box size="1 2 1"/>
+                <box size="1 1 2"/>
             </geometry>
         </collision>
     </link>
+    <!-- Joint for placing second floor on top of first floor, horizontal movement -->
     <joint name="firstFloor_to_secondFloor" type="prismatic">
-        <origin xyz="0 0.25 0" rpy="0 0 0"/>
+        <origin xyz="0 0 2" rpy="0 0 0"/> <!-- Placing second floor above the first floor -->
         <parent link="firstFloor"/>
         <child link="secondFloor"/>
-        <axis xyz="1 0 0"/> <!-- Allows horizontal motion along the x-axis -->
+        <axis xyz="1 0 0"/> <!-- Horizontal movement along the x-axis -->
         <limit lower="-1.0" upper="1.0" effort="1000" velocity="1.0"/>
     </joint>
     <link name="secondFloor">
         <visual>
-            <origin xyz="0 0 0" rpy="0 0 0"/>
+            <origin xyz="0 0 1" rpy="0 0 0"/>
             <geometry>
-                <box size="1 2 1"/>
+                <box size="1 1 2"/>
             </geometry>
-            <material name="magenta"/>
+            <material name="green"/> <!-- Color changed to green -->
+        </visual>
+        <collision>
+            <origin xyz="0 0 1" rpy="0 0 0"/>
+            <geometry>
+                <box size="1 1 2"/>
+            </geometry>
+        </collision>
+    </link>
+    <!-- Joint for placing third floor on top of second floor, horizontal movement -->
+    <joint name="secondFloor_to_thirdFloor" type="prismatic">
+        <origin xyz="0 0 2" rpy="0 0 0"/> <!-- Placing third floor above the second floor -->
+        <parent link="secondFloor"/>
+        <child link="thirdFloor"/>
+        <axis xyz="1 0 0"/> <!-- Horizontal movement along the x-axis -->
+        <limit lower="-1.0" upper="1.0" effort="1000" velocity="1.0"/>
+    </joint>
+    <link name="thirdFloor">
+        <visual>
+            <origin xyz="0 0 1" rpy="0 0 0"/>
+            <geometry>
+                <box size="1 1 2"/>
+            </geometry>
+            <material name="blue"/> <!-- Color changed to blue -->
+        </visual>
+        <collision>
+            <origin xyz="0 0 1" rpy="0 0 0"/>
+            <geometry>
+                <box size="1 1 2"/>
+            </geometry>
+        </collision>
+    </link>
+    <!-- Joint for placing fourth floor on top of third floor, horizontal movement -->
+    <joint name="thirdFloor_to_fourthFloor" type="prismatic">
+        <origin xyz="0 0 2" rpy="0 0 0"/> <!-- Placing fourth floor above the third floor -->
+        <parent link="thirdFloor"/>
+        <child link="fourthFloor"/>
+        <axis xyz="1 0 0"/> <!-- Horizontal movement along the x-axis -->
+        <limit lower="-1.0" upper="1.0" effort="1000" velocity="1.0"/>
+    </joint>
+    <link name="fourthFloor">
+        <visual>
+            <origin xyz="0 0 1" rpy="0 0 0"/>
+            <geometry>
+                <box size="1 1  2"/>
+            </geometry>
+            <material name="yellow"/> <!-- Color changed to yellow -->
         </visual>
         <collision>
             <origin xyz="0 0 0" rpy="0 0 0"/>
             <geometry>
-                <box size="1 2 1"/>
+                <box size="1 1 2"/>
             </geometry>
         </collision>
     </link>
-    <joint name="secondFloor_to_thirdFloor" type="prismatic">
-        <origin xyz="0 0.25 0" rpy="0 0 0"/>
-        <parent link="secondFloor"/>
-        <child link="thirdFloor"/>
-        <axis xyz="1 0 0"/> <!-- Allows horizontal motion along the x-axis -->
+    <!-- Joint for placing fifth floor on top of fourth floor, horizontal movement -->
+    <joint name="fourthFloor_to_fifthFloor" type="prismatic">
+        <origin xyz="0 0 2" rpy="0 0 0"/> <!-- Placing fifth floor above the fourth floor -->
+        <parent link="fourthFloor"/>
+        <child link="fifthFloor"/>
+        <axis xyz="1 0 0"/> <!-- Horizontal movement along the x-axis -->
         <limit lower="-1.0" upper="1.0" effort="1000" velocity="1.0"/>
     </joint>
-    <link name="thirdFloor">
+    <link name="fifthFloor">
         <visual>
-            <origin xyz="0 0 0" rpy="0 0 0"/>
+            <origin xyz="0 0 1" rpy="0 0 0"/>
             <geometry>
-                <box size="1 2 1"/>
+                <box size="1 1 2 "/>
             </geometry>
-            <material name="magenta"/>
+            <material name="cyan"/> <!-- Color changed to cyan -->
         </visual>
         <collision>
             <origin xyz="0 0 0" rpy="0 0 0"/>
             <geometry>
-                <box size="1 2 1"/>
-            </geometry>
-        </collision>
-    </link>
-    <joint name="thirdFloor_to_fourthFloor" type="prismatic">
-        <origin xyz="0 0.25 0" rpy="0 0 0"/>
-        <parent link="thirdFloor"/>
-        <child link="fourthFloor"/>
-        <axis xyz="1 0 0"/> <!-- Allows horizontal motion along the x-axis -->
-        <limit lower="-1.0" upper="1.0" effort="1000" velocity="1.0"/>
-    </joint>
-    <link name="fourthFloor">
-        <visual>
-            <origin xyz="0 0 0" rpy="0 0 0"/>
-            <geometry>
-                <box size="1 2 1"/>
-            </geometry>
-            <material name="magenta"/>
-        </visual>
-        <collision>
-            <origin xyz="0 0 0" rpy="0 0 0"/>
-            <geometry>
-                <box size="1 2 1"/>
-            </geometry>
-        </collision>
-    </link>
-    <joint name="fourthFloor_to_fifthFloor" type="prismatic">
-        <origin xyz="0 0.25 0" rpy="0 0 0"/>
-        <parent link="fourthFloor"/>
-        <child link="fifthFloor"/>
-        <axis xyz="1 0 0"/> <!-- Allows horizontal motion along the x-axis -->
-        <limit lower="-1.0" upper="1.0" effort="1000" velocity="1.0"/>
-    </joint>
-    <link name="fifthFloor">
-        <visual>
-            <origin xyz="0 0 0" rpy="0 0 0"/>
-            <geometry>
-                <box size="1 2 1"/>
-            </geometry>
-            <material name="magenta"/>
-        </visual>
-        <collision>
-            <origin xyz="0 0 0" rpy="0 0 0"/>
-            <geometry>
-                <box size="1 2 1"/>
+                <box size="1 1 2"/>
             </geometry>
         </collision>

Commit message: record

File: urdf/digitwin.urdf.xacro (robot description, xacro)
@@ -1,2 +1,3 @@
+<?xml version="1.0"?>
 <robot xmlns:xacro="http://www.ros.org/wiki/xacro" name="twin">
     <material name="gray">
@@ -54,5 +55,5 @@
         <child link="firstFloor"/>
         <axis xyz="1 0 0"/> <!-- Horizontal movement along the x-axis -->
-        <limit lower="-1.0" upper="1.0" effort="1000" velocity="1.0"/>
+        <limit lower="-0.1" upper="0.1" effort="1000" velocity="1.0"/>
     </joint>
     <link name="firstFloor">
@@ -77,5 +78,5 @@
         <child link="secondFloor"/>
         <axis xyz="1 0 0"/> <!-- Horizontal movement along the x-axis -->
-        <limit lower="-1.0" upper="1.0" effort="1000" velocity="1.0"/>
+        <limit lower="-0.1" upper="0.1" effort="1000" velocity="1.0"/>
     </joint>
     <link name="secondFloor">
@@ -100,5 +101,5 @@
         <child link="thirdFloor"/>
         <axis xyz="1 0 0"/> <!-- Horizontal movement along the x-axis -->
-        <limit lower="-1.0" upper="1.0" effort="1000" velocity="1.0"/>
+        <limit lower="-0.1" upper="0.1" effort="1000" velocity="1.0"/>
     </joint>
     <link name="thirdFloor">
@@ -123,5 +124,5 @@
         <child link="fourthFloor"/>
         <axis xyz="1 0 0"/> <!-- Horizontal movement along the x-axis -->
-        <limit lower="-1.0" upper="1.0" effort="1000" velocity="1.0"/>
+        <limit lower="-0.1" upper="0.1" effort="1000" velocity="1.0"/>
     </joint>
     <link name="fourthFloor">
@@ -146,5 +147,5 @@
         <child link="fifthFloor"/>
         <axis xyz="1 0 0"/> <!-- Horizontal movement along the x-axis -->
-        <limit lower="-1.0" upper="1.0" effort="1000" velocity="1.0"/>
+        <limit lower="-0.1" upper="0.1" effort="1000" velocity="1.0"/>
     </joint>
     <link name="fifthFloor">
